Commit message: Copy UR launch file format

File: robot_specific_config/abb_irb1200_5_90_moveit_config/config/abb_irb1200_5_90_macro.srdf.xacro (robot description, xacro)
@@ -1,13 +1,5 @@
 <?xml version="1.0" encoding="utf-8"?>
-<!--This does not replace URDF, and is not an extension of URDF.
-    This is a format for representing semantic information about the robot structure.
-    A URDF file must exist for this robot as well, where the joints and the links that are referenced are defined
--->
-<robot name="abb_irb1200_5_90">
-    <!--GROUPS: Representation of a set of joints and links. This can be useful for specifying DOF to plan for, defining arms, end effectors, etc-->
-    <!--LINKS: When a link is specified, the parent joint of that link (if it exists) is automatically included-->
-    <!--JOINTS: When a joint is specified, the child link of that joint (which will always exist) is automatically included-->
-    <!--CHAINS: When a chain is specified, all the links along the chain (including endpoints) are included in the group. Additionally, all the joints that are parents to included links are also included. This means that joints along the chain and the parent joint of the base link are included in the group-->
-    <!--SUBGROUPS: Groups can also be formed by referencing to already defined group names-->
+<robot xmlns:xacro="http://wiki.ros.org/xacro">
+  <xacro:macro name="abb_irb1200_5_90_srdf">
     <group name="manipulator">
         <chain base_link="base_link" tip_link="tool0" />
@@ -35,3 +27,4 @@
     <disable_collisions link1="link_4" link2="link_5" reason="Adjacent" />
     <disable_collisions link1="link_5" link2="link_6" reason="Adjacent" />
+  </xacro:macro>
 </robot>
